File: reverb.brd (EAGLE design)
At the start: 152.4 x 25.4 mm, 59 parts, among them IC2 TL074, IC2_EQ1 NE5532, IC4_DRV_RCVR TL072, T1 2N3904

Commit message: oops, the +12V needed to be +12_B
should really rename that one later
Connections:
- removed net +12V: BLND.1, LED.A
- net +12V_B: now also BLND.1, LED.A
Routing:
- net +12V: track 27.7 -> 0.00 mm
- net +12V_B: track 128.7 -> 156.2 mm, vias 0 -> 1
Changed lines of the file:
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@@
 <grid distance="0.0125" unitdist="inch" unit="inch" style="lines" multiple="1" display="no" altdistance="0.00125" altunitdist="inch" altunit="inch"/>
 <layers>
-<layer number="1" name="Top" color="4" fill="1" visible="no" active="yes"/>
+<layer number="1" name="Top" color="4" fill="1" visible="yes" active="yes"/>
 <layer number="2" name="Route2" color="1" fill="3" visible="no" active="no"/>
 <layer number="3" name="Route3" color="4" fill="3" visible="no" active="no"/>
 <layer number="14" name="Route14" color="1" fill="6" visible="no" active="no"/>
 <layer number="15" name="Route15" color="4" fill="6" visible="no" active="no"/>
-<layer number="16" name="Bottom" color="1" fill="1" visible="no" active="yes"/>
-<layer number="17" name="Pads" color="2" fill="1" visible="no" active="yes"/>
-<layer number="18" name="Vias" color="2" fill="1" visible="no" active="yes"/>
-<layer number="19" name="Unrouted" color="6" fill="1" visible="no" active="yes"/>
-<layer number="20" name="Dimension" color="15" fill="1" visible="no" active="yes"/>
-<layer number="21" name="tPlace" color="7" fill="1" visible="no" active="yes"/>
-<layer number="22" name="bPlace" color="7" fill="1" visible="no" active="yes"/>
+<layer number="16" name="Bottom" color="1" fill="1" visible="yes" active="yes"/>
+<layer number="17" name="Pads" color="2" fill="1" visible="yes" active="yes"/>
+<layer number="18" name="Vias" color="2" fill="1" visible="yes" active="yes"/>
+<layer number="19" name="Unrouted" color="6" fill="1" visible="yes" active="yes"/>
+<layer number="20" name="Dimension" color="15" fill="1" visible="yes" active="yes"/>
+<layer number="21" name="tPlace" color="7" fill="1" visible="yes" active="yes"/>
+<layer number="22" name="bPlace" color="7" fill="1" visible="yes" active="yes"/>
 <layer number="23" name="tOrigins" color="15" fill="1" visible="no" active="yes"/>
 <layer number="24" name="bOrigins" color="15" fill="1" visible="no" active="yes"/>
-<layer number="25" name="tNames" color="7" fill="1" visible="no" active="yes"/>
+<layer number="25" name="tNames" color="7" fill="1" visible="yes" active="yes"/>
 <layer number="26" name="bNames" color="7" fill="1" visible="no" active="yes"/>
 <layer number="27" name="tValues" color="7" fill="1" visible="yes" active="yes"/>
@@
 <wire x1="59.8931" y1="18.415" x2="58.8262" y2="19.4819" width="0.6096" layer="1"/>
 <wire x1="58.8262" y1="19.4819" x2="54.8131" y2="19.4819" width="0.6096" layer="1"/>
-<wire x1="54.8131" y1="19.4819" x2="54.178" y2="20.117" width="0.6096" layer="1"/>
-<wire x1="54.178" y1="20.117" x2="26.2508" y2="20.117" width="0.6096" layer="1"/>
-<wire x1="26.2508" y1="20.117" x2="22.8728" y2="23.495" width="0.6096" layer="1"/>
+<wire x1="54.8131" y1="19.4819" x2="54.178" y2="20.4345" width="0.6096" layer="1"/>
+<wire x1="54.178" y1="20.4345" x2="26.2508" y2="20.4345" width="0.6096" layer="1"/>
+<wire x1="26.2508" y1="20.4345" x2="26.047665625" y2="20.618540625" width="0.6096" layer="1"/>
+<wire x1="26.047665625" y1="20.618540625" x2="22.8728" y2="23.495" width="0.6096" layer="1"/>
 <wire x1="60.96" y1="15.875" x2="60.96" y2="17.5515" width="0.6096" layer="1"/>
 <wire x1="93.345" y1="8.89" x2="94.4119" y2="8.89" width="0.6096" layer="1"/>
@@
 <wire x1="90.17" y1="7.62" x2="91.0081" y2="7.62" width="0.6096" layer="16"/>
 <wire x1="91.0081" y1="7.62" x2="92.2781" y2="8.89" width="0.6096" layer="16"/>
+<contactref element="LED" pad="A"/>
+<contactref element="BLND" pad="1"/>
+<wire x1="28.8925" y1="23.495" x2="28.8925" y2="23.463375" width="0.4064" layer="1"/>
+<wire x1="28.8925" y1="23.463375" x2="26.047665625" y2="20.618540625" width="0.6096" layer="1"/>
+<wire x1="26.2508" y1="20.4345" x2="25.832" y2="20.4345" width="0.4064" layer="1"/>
+<wire x1="25.832" y1="20.4345" x2="20.6375" y2="15.24" width="0.6096" layer="1"/>
+<wire x1="20.6375" y1="15.24" x2="20.6375" y2="9.525" width="0.6096" layer="1"/>
+<wire x1="20.6375" y1="9.525" x2="22.225" y2="7.9375" width="0.6096" layer="1"/>
+<via x="22.225" y="7.9375" extent="1-16" drill="0.6" shape="square"/>
+<wire x1="22.225" y1="7.9375" x2="23.1775" y2="7.9375" width="0.6096" layer="16"/>
+<wire x1="23.1775" y1="7.9375" x2="27.94" y2="3.175" width="0.6096" layer="16"/>
 </signal>
 <signal name="-12V_B" class="1">
@@
 <wire x1="60.96" y1="10.795" x2="61.39175" y2="10.36325" width="0.6096" layer="16"/>
 </signal>
-<signal name="+12V" class="1">
-<contactref element="BLND" pad="1"/>
-<contactref element="LED" pad="A"/>
-<wire x1="28.8925" y1="23.495" x2="27.9907" y2="23.1775" width="0.6096" layer="16"/>
-<wire x1="27.94" y1="3.175" x2="26.8731" y2="3.175" width="0.6096" layer="16"/>
-<wire x1="26.8731" y1="3.175" x2="20.7864" y2="10.2142" width="0.6096" layer="16"/>
-<wire x1="20.7864" y1="10.2142" x2="20.7864" y2="17.2432" width="0.6096" layer="16"/>
-<wire x1="20.7864" y1="17.2432" x2="27.9907" y2="23.1775" width="0.6096" layer="16"/>
-</signal>
 <signal name="GND" class="2">
