File: reverb.sch (EAGLE design)
At the start: 59 parts, among them IC2 TL074, IC2_EQ1 NE5532, IC4_DRV_RCVR TL072, T1 2N3904

Commit message: moved some stuff around.. might need to hook up some gnds still
Parts:
- ATTN, BLND: value (none) -> 50K
- EQ: value (none) -> 10K
- SWITCH: value (none) -> XFADE_OR_REVERB
- renumbered ATTN_50K to ATTN, AUDIO_IN to IN, AUDIO_OUT to OUT, BLEND_50K to BLND, CV_IN to CV, TILT_EQ10K to EQ, XFADE_REV_SWITCH to SWITCH
Changed lines of the file:
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@@
 <part name="R34" library="TomW" deviceset="R-EU_" device="STANDARD_RESISTOR" value="100k"/>
 <part name="SUPPLY9" library="supply2" deviceset="GND" device=""/>
-<part name="TILT_EQ10K" library="pinhead" deviceset="PINHD-1X3" device=""/>
-<part name="BLEND_50K" library="pinhead" deviceset="PINHD-1X3" device=""/>
-<part name="ATTN_50K" library="pinhead" deviceset="PINHD-1X3" device=""/>
-<part name="AUDIO_IN" library="pinhead" deviceset="PINHD-1X2" device=""/>
-<part name="AUDIO_OUT" library="pinhead" deviceset="PINHD-1X2" device=""/>
+<part name="EQ" library="pinhead" deviceset="PINHD-1X3" device="" value="10K"/>
+<part name="BLND" library="pinhead" deviceset="PINHD-1X3" device="" value="50K"/>
+<part name="ATTN" library="pinhead" deviceset="PINHD-1X3" device="" value="50K"/>
+<part name="IN" library="pinhead" deviceset="PINHD-1X2" device=""/>
+<part name="OUT" library="pinhead" deviceset="PINHD-1X2" device=""/>
 <part name="XFADE_IN" library="pinhead" deviceset="PINHD-1X2" device=""/>
-<part name="XFADE_REV_SWITCH" library="pinhead" deviceset="PINHD-1X2" device=""/>
-<part name="CV_IN" library="pinhead" deviceset="PINHD-1X2" device=""/>
+<part name="SWITCH" library="pinhead" deviceset="PINHD-1X2" device="" value="XFADE_OR_REVERB"/>
+<part name="CV" library="pinhead" deviceset="PINHD-1X2" device=""/>
 <part name="J1" library="con-amp" deviceset="MTA04-156" device=""/>
 </parts>
@@
 <instance part="R34" gate="G$1" x="111.76" y="27.94" rot="R90"/>
 <instance part="SUPPLY9" gate="GND" x="111.76" y="17.78"/>
-<instance part="TILT_EQ10K" gate="A" x="20.32" y="20.32"/>
-<instance part="BLEND_50K" gate="A" x="33.02" y="58.42" rot="MR0"/>
-<instance part="ATTN_50K" gate="A" x="-27.94" y="81.28" rot="MR0"/>
-<instance part="AUDIO_IN" gate="G$1" x="-93.98" y="101.6" rot="MR0"/>
-<instance part="AUDIO_OUT" gate="G$1" x="129.54" y="96.52" rot="R180"/>
+<instance part="EQ" gate="A" x="20.32" y="20.32"/>
+<instance part="BLND" gate="A" x="33.02" y="58.42" rot="MR0"/>
+<instance part="ATTN" gate="A" x="-27.94" y="81.28" rot="MR0"/>
+<instance part="IN" gate="G$1" x="-93.98" y="101.6" rot="MR0"/>
+<instance part="OUT" gate="G$1" x="129.54" y="96.52" rot="R180"/>
 <instance part="XFADE_IN" gate="G$1" x="55.88" y="30.48" rot="MR0"/>
-<instance part="XFADE_REV_SWITCH" gate="G$1" x="68.58" y="7.62" rot="MR0"/>
-<instance part="CV_IN" gate="G$1" x="-38.1" y="101.6" rot="R180"/>
+<instance part="SWITCH" gate="G$1" x="68.58" y="7.62" rot="MR0"/>
+<instance part="CV" gate="G$1" x="-38.1" y="101.6" rot="R180"/>
 <instance part="IC2_EQ1" gate="P" x="-60.96" y="-40.64"/>
 <instance part="IC2" gate="P" x="-53.34" y="-40.64"/>
@@
 <wire x1="45.72" y1="48.26" x2="45.72" y2="50.8" width="0.1524" layer="91"/>
 <wire x1="45.72" y1="50.8" x2="45.72" y2="55.88" width="0.1524" layer="91"/>
-<pinref part="BLEND_50K" gate="A" pin="3"/>
+<pinref part="BLND" gate="A" pin="3"/>
 <wire x1="45.72" y1="55.88" x2="35.56" y2="55.88" width="0.1524" layer="91"/>
 </segment>
@@
 <wire x1="-15.24" y1="73.66" x2="-15.24" y2="76.2" width="0.1524" layer="91"/>
 <wire x1="-15.24" y1="76.2" x2="-15.24" y2="78.74" width="0.1524" layer="91"/>
-<pinref part="ATTN_50K" gate="A" pin="3"/>
+<pinref part="ATTN" gate="A" pin="3"/>
 <wire x1="-15.24" y1="78.74" x2="-25.4" y2="78.74" width="0.1524" layer="91"/>
 </segment>
@@
 <wire x1="-27.94" y1="101.6" x2="-20.32" y2="101.6" width="0.1524" layer="91"/>
 <pinref part="SUPPLY13" gate="GND" pin="GND"/>
-<pinref part="CV_IN" gate="G$1" pin="2"/>
+<pinref part="CV" gate="G$1" pin="2"/>
 <wire x1="-27.94" y1="101.6" x2="-35.56" y2="101.6" width="0.1524" layer="91"/>
 </segment>
@@
 <pinref part="SUPPLY20" gate="GND" pin="GND"/>
 <wire x1="154.94" y1="96.52" x2="147.32" y2="96.52" width="0.1524" layer="91"/>
-<pinref part="AUDIO_OUT" gate="G$1" pin="2"/>
+<pinref part="OUT" gate="G$1" pin="2"/>
 <wire x1="147.32" y1="96.52" x2="132.08" y2="96.52" width="0.1524" layer="91"/>
 </segment>
@@
 <wire x1="-76.2" y1="93.98" x2="-76.2" y2="99.06" width="0.1524" layer="91"/>
 <wire x1="-76.2" y1="99.06" x2="-76.2" y2="101.6" width="0.1524" layer="91"/>
-<pinref part="AUDIO_IN" gate="G$1" pin="2"/>
+<pinref part="IN" gate="G$1" pin="2"/>
 <wire x1="-76.2" y1="101.6" x2="-91.44" y2="101.6" width="0.1524" layer="91"/>
 </segment>
@@
 <wire x1="45.72" y1="66.04" x2="45.72" y2="60.96" width="0.1524" layer="91"/>
 <wire x1="45.72" y1="60.96" x2="38.1" y2="60.96" width="0.1524" layer="91"/>
-<pinref part="BLEND_50K" gate="A" pin="1"/>
+<pinref part="BLND" gate="A" pin="1"/>
 <wire x1="38.1" y1="60.96" x2="35.56" y2="60.96" width="0.1524" layer="91"/>
 </segment>
@@
 <pinref part="R33" gate="G$1" pin="2"/>
 <wire x1="55.88" y1="58.42" x2="55.88" y2="63.5" width="0.1524" layer="91"/>
-<pinref part="BLEND_50K" gate="A" pin="2"/>
+<pinref part="BLND" gate="A" pin="2"/>
 <wire x1="50.8" y1="58.42" x2="35.56" y2="58.42" width="0.1524" layer="91"/>
 </segment>
@@
 <wire x1="147.32" y1="91.44" x2="147.32" y2="78.74" width="0.1524" layer="91"/>
 <wire x1="147.32" y1="91.44" x2="147.32" y2="93.98" width="0.1524" layer="91"/>
-<pinref part="AUDIO_OUT" gate="G$1" pin="1"/>
+<pinref part="OUT" gate="G$1" pin="1"/>
 <wire x1="147.32" y1="93.98" x2="132.08" y2="93.98" width="0.1524" layer="91"/>
 </segment>
@@
 <wire x1="-10.16" y1="83.82" x2="-15.24" y2="83.82" width="0.1524" layer="91"/>
 <wire x1="-15.24" y1="83.82" x2="-15.24" y2="81.28" width="0.1524" layer="91"/>
-<pinref part="ATTN_50K" gate="A" pin="2"/>
+<pinref part="ATTN" gate="A" pin="2"/>
 <wire x1="-15.24" y1="81.28" x2="-25.4" y2="81.28" width="0.1524" layer="91"/>
 </segment>
@@
 <wire x1="-20.32" y1="63.5" x2="-15.24" y2="63.5" width="0.1524" layer="91"/>
 <wire x1="-27.94" y1="96.52" x2="-27.94" y2="91.44" width="0.1524" layer="91"/>
-<pinref part="ATTN_50K" gate="A" pin="1"/>
+<pinref part="ATTN" gate="A" pin="1"/>
 <wire x1="-20.32" y1="83.82" x2="-25.4" y2="83.82" width="0.1524" layer="91"/>
 <junction x="-20.32" y="83.82"/>
 <wire x1="-27.94" y1="96.52" x2="-27.94" y2="99.06" width="0.1524" layer="91"/>
-<pinref part="CV_IN" gate="G$1" pin="1"/>
+<pinref part="CV" gate="G$1" pin="1"/>
 <wire x1="-27.94" y1="99.06" x2="-35.56" y2="99.06" width="0.1524" layer="91"/>
 </segment>
@@
 <wire x1="-76.2" y1="119.38" x2="-71.12" y2="119.38" width="0.1524" layer="91"/>
 <wire x1="-76.2" y1="119.38" x2="-76.2" y2="104.14" width="0.1524" layer="91"/>
-<pinref part="AUDIO_IN" gate="G$1" pin="1"/>
+<pinref part="IN" gate="G$1" pin="1"/>
 <wire x1="-76.2" y1="104.14" x2="-91.44" y2="104.14" width="0.1524" layer="91"/>
 </segment>
@@
 <wire x1="2.54" y1="27.94" x2="2.54" y2="25.4" width="0.1524" layer="91"/>
 <wire x1="2.54" y1="25.4" x2="2.54" y2="22.86" width="0.1524" layer="91"/>
-<pinref part="TILT_EQ10K" gate="A" pin="1"/>
+<pinref part="EQ" gate="A" pin="1"/>
 <wire x1="2.54" y1="22.86" x2="17.78" y2="22.86" width="0.1524" layer="91"/>
 </segment>
@@
 <junction x="2.54" y="7.62"/>
 <wire x1="2.54" y1="12.7" x2="2.54" y2="17.78" width="0.1524" layer="91"/>
-<pinref part="TILT_EQ10K" gate="A" pin="3"/>
+<pinref part="EQ" gate="A" pin="3"/>
 <wire x1="2.54" y1="17.78" x2="17.78" y2="17.78" width="0.1524" layer="91"/>
 </segment>
@@
 <wire x1="10.16" y1="-12.7" x2="7.62" y2="-12.7" width="0.1524" layer="91"/>
 <wire x1="7.62" y1="-12.7" x2="7.62" y2="-2.54" width="0.1524" layer="91"/>
-<pinref part="TILT_EQ10K" gate="A" pin="2"/>
+<pinref part="EQ" gate="A" pin="2"/>
 <wire x1="-2.54" y1="20.32" x2="17.78" y2="20.32" width="0.1524" layer="91"/>
 </segment>
@@
 <wire x1="81.28" y1="7.62" x2="73.66" y2="7.62" width="0.1524" layer="91"/>
 <label x="83.82" y="7.62" size="1.778" layer="95"/>
-<pinref part="XFADE_REV_SWITCH" gate="G$1" pin="2"/>
+<pinref part="SWITCH" gate="G$1" pin="2"/>
 <wire x1="73.66" y1="7.62" x2="71.12" y2="7.62" width="0.1524" layer="91"/>
 </segment>
@@
 <pinref part="XFADE_IN" gate="G$1" pin="1"/>
 <wire x1="71.12" y1="33.02" x2="58.42" y2="33.02" width="0.1524" layer="91"/>
-<pinref part="XFADE_REV_SWITCH" gate="G$1" pin="1"/>
+<pinref part="SWITCH" gate="G$1" pin="1"/>
 <wire x1="71.12" y1="10.16" x2="78.74" y2="10.16" width="0.1524" layer="91"/>
 <wire x1="78.74" y1="10.16" x2="78.74" y2="33.02" width="0.1524" layer="91"/>

Commit message: everything is hooked up and not overlapping!
Parts:
- renumbered LED1 to LED
Changed lines of the file:
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@@
 <part name="SUPPLY15" library="supply2" deviceset="GND" device=""/>
 <part name="R17" library="TomW" deviceset="VERT-RESIST1" device="" value="47k"/>
-<part name="LED1" library="TomW" deviceset="LED" device="3MM" value="3mm Superbright"/>
+<part name="LED" library="TomW" deviceset="LED" device="3MM" value="3mm Superbright"/>
 <part name="SUPPLY23" library="supply2" deviceset="GND" device=""/>
 <part name="IC2" library="linear" deviceset="TL074" device="P" value="TL074"/>
@@
 <instance part="SUPPLY15" gate="GND" x="-15.24" y="71.12"/>
 <instance part="R17" gate="G$1" x="7.62" y="63.5"/>
-<instance part="LED1" gate="G$1" x="73.66" y="109.22"/>
+<instance part="LED" gate="G$1" x="73.66" y="109.22"/>
 <instance part="SUPPLY23" gate="GND" x="73.66" y="55.88"/>
 <instance part="IC2" gate="D" x="119.38" y="78.74"/>
@@
 <segment>
 <pinref part="SUPPLY17" gate="+12V" pin="+12V"/>
-<pinref part="LED1" gate="G$1" pin="A"/>
+<pinref part="LED" gate="G$1" pin="A"/>
 <wire x1="73.66" y1="111.76" x2="73.66" y2="116.84" width="0.1524" layer="91"/>
 </segment>
@@
 <segment>
 <pinref part="LDR1" gate="G$1" pin="LED+"/>
-<pinref part="LED1" gate="G$1" pin="C"/>
+<pinref part="LED" gate="G$1" pin="C"/>
 <wire x1="73.66" y1="104.14" x2="73.66" y2="96.52" width="0.1524" layer="91"/>
 </segment>

Commit message: oops, the +12V needed to be +12_B
should really rename that one later
Connections:
- removed net +12V: BLND.1, LED.A
- net +12V_B: now also BLND.1, LED.A
Changed lines of the file:
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@@
-</segment>
-</net>
-<net name="+12V" class="1">
-<segment>
-<pinref part="SUPPLY16" gate="+12V" pin="+12V"/>
-<wire x1="45.72" y1="68.58" x2="45.72" y2="66.04" width="0.1524" layer="91"/>
-<wire x1="45.72" y1="66.04" x2="45.72" y2="60.96" width="0.1524" layer="91"/>
-<wire x1="45.72" y1="60.96" x2="38.1" y2="60.96" width="0.1524" layer="91"/>
-<pinref part="BLND" gate="A" pin="1"/>
-<wire x1="38.1" y1="60.96" x2="35.56" y2="60.96" width="0.1524" layer="91"/>
-</segment>
-<segment>
-<pinref part="SUPPLY17" gate="+12V" pin="+12V"/>
-<pinref part="LED" gate="G$1" pin="A"/>
-<wire x1="73.66" y1="111.76" x2="73.66" y2="116.84" width="0.1524" layer="91"/>
 </segment>
 </net>
@@
 <label x="-58.42" y="-25.4" size="1.778" layer="95"/>
 </segment>
-</net>
+<segment>
+<pinref part="SUPPLY17" gate="+12V" pin="+12V"/>
+<pinref part="LED" gate="G$1" pin="A"/>
+<wire x1="73.66" y1="111.76" x2="73.66" y2="116.84" width="0.1524" layer="91"/>
+</segment>
+<segment>
+<pinref part="SUPPLY16" gate="+12V" pin="+12V"/>
+<wire x1="45.72" y1="68.58" x2="45.72" y2="66.04" width="0.1524" layer="91"/>
+<wire x1="45.72" y1="66.04" x2="45.72" y2="60.96" width="0.1524" layer="91"/>
+<wire x1="45.72" y1="60.96" x2="38.1" y2="60.96" width="0.1524" layer="91"/>
+<pinref part="BLND" gate="A" pin="1"/>
+<wire x1="38.1" y1="60.96" x2="35.56" y2="60.96" width="0.1524" layer="91"/>
+</segment>
+</net>
